File: HW2+HW3/ME 433/galePCB.brd (EAGLE design)
At the start: 50 x 50 mm, 22 parts, among them J4 USB-MB-H

Commit message: making gerber files
Parts:
- moved C4 1.27 mm to (17.8, 43.2)
- moved U$4 0.82 mm to (15.8, 47.8), flipped to the bottom
- moved R8 0.67 mm to (21.5, 1.94)
- moved R6 0.67 mm to (11.4, 7.02)
- moved GRN 0.46 mm to (3.00, 11.4)
- moved R7 0.44 mm to (7.69, 6.78)
- moved J4 0.10 mm to (3.88, 44.4)
Connections:
- net +5V: now also C4.1, U$2.2, U$4.2
- net VBUS: no longer C4.1, U$2.2, U$4.2
Routing:
- net +5V: track 25.5 -> 81.7 mm, vias 0 -> 2
- net A0: track 2.54 -> 21.4 mm
- net VBUS: track 20.0 -> 7.64 mm
- net D+: track 27.5 -> 37.6 mm, vias 0 -> 1
- net +3V3: track 120.8 -> 120.2 mm
- net A4/LED: track 34.9 -> 34.3 mm
- net PGC: vias 0 -> 1
