File: HW2+HW3/ME 433/galePCB2.sch (EAGLE design)
At the start: 19 parts, among them J4 USB-MB-H

Commit message: making gerber files
Parts:
- removed R1, R2: 330, myPCB:R-US_0309/12
- removed R3, R4: 10K, myPCB:R-US_0309/12
- removed RED_LED: (no value), myPCB:LED3MM
- removed U$3: CRYSTAL_RES, myPCB:CRYSTAL_RES
- added 8MHZ: (no value), myPCB:M03PTH
- added J2: (no value), myPCB:M08
- added PICKIT: (no value), myPCB:M05PTH
- added R5, R6: 10k, myPCB:R-US_0207/10
- added R7, R8: 330, myPCB:R-US_0207/10
- added RED: (no value), myPCB:LED3MM
- added U$4: SLIDESWITCH, myPCB:SLIDESWITCH
- C1: value 10uF -> +10uF-
- C3: value (none) -> 0.1 uF
- J1: device myPCB:M06POLAR -> myPCB:M08
- U$1: value PIC32 -> PIC32MX250F128B
- renumbered GREEN_LED to GRN
Connections:
- removed net BUTTON: R4.1, U$1.11.SOSCI, USER.3
- removed net N$4: GRN.A, U$1.12.SOSCO
- removed net N$7: C5.2, C6.1
- removed net N$8: GRN.C, R1.2
- new net +5V: C4.1, J2.2, U$1.15.VBUS, U$2.2.VIN, U$4.OUT1
- new net A4/LED: GRN.A, J1.3, U$1.12.SOSCO
- new net B13: J2.6, U$1.24.AN11
- new net B14: J2.7, U$1.25.CVREF
- new net B15: J2.8, U$1.26.AN9
- new net B4/USER: J1.4, R6.1, U$1.11.SOSCI, USER.3
- new net B7: J2.3, U$1.16.TDI
- new net B8: J2.4, U$1.17.TCK
- new net B9: J2.5, U$1.17.TDO
- new net USBID: J4.ID, U$1.14.TMS
- net +3V3: now also C5.1, C6.1, PICKIT.2, R5.2, R6.2, RED.A, U$2.3.VOUT; no longer C6.2, R3.2, R4.2, RED_LED.A
- net A0: now also J1.8
- net A1: now also J1.7
- net B2: now also J1.6
- net B3: now also J1.5
- net GND: now also 8MHZ.2, C5.2, C6.2, J1.1, J2.1, PICKIT.3, R7.1, R8.1; no longer J1.3, R1.1, R2.1
- net MCLR: now also PICKIT.1, R5.1; no longer J1.1, R3.1
- net N$2: now also 8MHZ.3
- net N$3: now also 8MHZ.1
- net N$5: now also R8.2, RED.C; no longer R2.2, RED_LED.C
- net N$6: now also GRN.C, R7.2; no longer C5.1, U$2.3.VOUT
- net PGC: now also PICKIT.5; no longer J1.5
- net PGD: now also PICKIT.4; no longer J1.4
- net VBUS: now also U$4.IN; no longer C4.1, U$1.15.VBUS, U$2.2.VIN
Other:
- moved on the sheet: C4, C5, C6, U$2
